Commit message: better viser setup

File: src/lerobot_3d/calibration/yam/yam_station_linear_4310_d405.urdf (robot description, URDF)
Before this commit: robot yam_station_linear_4310_d405, 21 links, 20 joints
Joints:
- joint right_base_joint: origin xyz=0 -0.61 0 rpy=0 0 0 -> xyz=0 0.61 0 rpy=0 0 0
- joint top_camera_joint: origin xyz=-0.16649488039785276 -0.3050000004052651 0.9543205295851617 rpy=-2.6179963071795864 -2.220446049250313e-16 -1.5708 -> xyz=-0.16649488039785276 0.3050000004052651 0.9543205295851617 rpy=-2.6179963071795864 -2.220446049250313e-16 -1.5708
